Commit message: Update hardware location.

File: src/rover_description/urdf/rover.urdf (robot description, URDF)
Before this commit: robot wave_rover, 3 links, 2 joints
Joints:
- joint laser_joint: origin xyz=0.12 0.0 0.10 rpy=0 0 0 -> xyz=0.12 0.0 0.240 rpy=0 0 0

Commit message: update yaml.

File: src/rover_description/urdf/rover.urdf (robot description, URDF)
Before this commit: robot wave_rover, 3 links, 2 joints
Joints:
- joint imu_joint: origin xyz=0.0 0.0 0.05 rpy=0 0 0 -> xyz=0.0381 0.00635 0.0300 rpy=0 0 0
- joint laser_joint: origin xyz=0.12 0.0 0.240 rpy=0 0 0 -> xyz=-0.0381 0.00635 0.1524 rpy=0 0 0
